File: KeyboardBase/Column.kicad_sch (KiCad schematic)
At the start: 1 part, among them J1201 Conn_01x06

Commit message: fix pin label, reduce column keys to 4
Connections:
- net Reset_ROW renamed ~{Reset_ROW}
Other:
- sheet SelectorDaisy ports: added ~{Reset}; removed Reset
Changed lines of the file:
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@@
 		)
 	)
-	(hierarchical_label "Reset"
+	(hierarchical_label "~{Reset}"
 		(shape input)
 		(at 62.23 78.74 180)
@@
 		)
 	)
-	(hierarchical_label "Reset_ROW"
+	(hierarchical_label "~{Reset_ROW}"
 		(shape input)
 		(at 86.36 45.72 180)
@@
 			)
 		)
-		(pin "Reset" input
-			(at 81.28 78.74 180)
-			(effects
-				(font
-					(size 1.27 1.27)
-				)
-				(justify left)
-			)
-		)
 		(pin "CLK" input
 			(at 81.28 83.82 180)
@@
 			(effects
 				(font
+					(size 1.27 1.27)
+				)
+				(justify left)
+			)
+		)
+		(pin "~{Reset}" input
+			(at 81.28 78.74 180)
+			(effects
+				(font

Commit message: change connector
Parts:
- J1201: Manufacturer Part number (none) -> 2005280060; Original (none) -> N; Purchase Link (none) -> https://www.digikey.com/en/products/detail/molex/2005280060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
Changed lines of the file:
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@@
 			)
 		)
-		(property "Description" "Generic connector, single row, 01x06, script generated (kicad-library-utils/schlib/autogen/connector/)"
+		(property "Description" "CONN FFC FPC BOTTOM 6POS 1MM R/A"
 			(at 99.06 50.8 0)
 			(effects
+				(font
+					(size 1.27 1.27)
+				)
+				(hide yes)
+			)
+		)
+		(property "Manufacturer Part number" "2005280060"
+			(at 99.06 50.8 0)
+			(effects
+				(font
+					(size 1.27 1.27)
+				)
+				(hide yes)
+			)
+		)
+		(property "Original" "N"
+			(at 99.06 50.8 0)
+			(effects
+				(font
+					(size 1.27 1.27)
+				)
+				(hide yes)
+			)
+		)
+		(property "Purchase Link" "https://www.digikey.com/en/products/detail/molex/2005280060/6099556"
+			(at 99.06 50.8 0)
+			(effects
