File: KeyboardBase/KeyboardBase.kicad_pcb (KiCad board)
At the start: 2 copper layers, 152.1 x 17.9 mm, 23 parts, among them J1001 Conn_01x06, J101 Conn_01x07, J1201 Conn_01x06, J1401 Conn_01x06, J201 Conn_01x06, J401 Conn_01x06, J601 Conn_01x06, J801 Conn_01x06, U101 74HC00, U1101 74HC00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

Commit message: fix circuit
Parts:
- added U102: 74HC00, Package_DFN_QFN:WQFN-14-1EP_2.5x2.5mm_P0.5mm_EP1.45x1.45mm, F.Cu at (83.2, 86.4)
- moved U101 4.05 mm to (82.5, 82.1), turned to 0 degrees
Connections:
- J1001 pad 5: /Column/Reset_ROW -> /Column/~{Reset_ROW}
- J101 pad 2: Reset -> Out
- J101 pad 3: CLK_COL -> ~{Any}
- J101 pad 4: Out -> ~{Reset}
- J101 pad 5: Vcc -> CLK_COL
- J101 pad 7: ~{Any} -> Vcc
- J1201 pad 5: /Column/Reset_ROW -> /Column/~{Reset_ROW}
- J1401 pad 5: /Column/Reset_ROW -> /Column/~{Reset_ROW}
- J201 pad 5: /Column/Reset_ROW -> /Column/~{Reset_ROW}
- J401 pad 5: /Column/Reset_ROW -> /Column/~{Reset_ROW}
- J601 pad 5: /Column/Reset_ROW -> /Column/~{Reset_ROW}
- J801 pad 5: /Column/Reset_ROW -> /Column/~{Reset_ROW}
- U101 pad 1: Reset -> CLK_COL
- U101 pad 10: CLK_COL -> Net-(U101-Pad10)
- U101 pad 2: Reset -> CLK_COL
- U101 pad 5: Net-(U101-Pad5) -> ~{Reset}
- U101 pad 6: /Column/Reset_ROW -> Net-(U101-Pad10)
- U101 pad 8: Net-(U101-Pad5) -> /Column/~{Reset_ROW}
- U101 pad 9: CLK_COL -> Net-(U101-Pad10)
- U1102 pad 1: Reset -> ~{Reset}
- U1302 pad 1: Reset -> ~{Reset}
- U1502 pad 1: Reset -> ~{Reset}
- U302 pad 1: Reset -> Vcc
- U302 pad 4: GND -> /Column/~{Init}
- U502 pad 1: Reset -> ~{Reset}
- U702 pad 1: Reset -> ~{Reset}
- U902 pad 1: Reset -> ~{Reset}
Routing:
- net ~{Reset}: vias 0 -> 14
- net Reset: vias 14 -> 0
- net Net-(U101-Pad10): vias 0 -> 2
- net GND: vias 87 -> 86
- net /Column/~{Reset_ROW}: vias 0 -> 14
- net /Column/~{Init}: vias 0 -> 2
- net /Column/Reset_ROW: vias 16 -> 0
Other:
- board size 152.1 x 17.9 mm -> 150.8 x 17.9 mm

Commit message: change connector
Parts:
- removed J101: Conn_01x07, Library:PinHeader 2.00mm 01x07 SMD
- added J102: 5023520701, Molex:CONN07_502352_MOL, F.Cu at (72.3, 83.3)
Routing:
- net ~{Any}: vias 16 -> 18
- net GND: vias 86 -> 93
Other:
- board size 150.8 x 17.9 mm -> 153.4 x 20.8 mm

Commit message: remove padding
Parts:
- moved J1401 6.00 mm to (203.5, 78.3)
- moved U1501 6.00 mm to (206.3, 84.8)
- moved U1502 6.00 mm to (202.2, 84.8)
- moved J1201 5.00 mm to (184.5, 78.3)
- moved U1301 5.00 mm to (187.3, 84.8)
- moved U1302 5.00 mm to (183.2, 84.8)
- moved J1001 4.00 mm to (165.5, 78.3)
- moved U1101 4.00 mm to (168.3, 84.8)
- moved U1102 4.00 mm to (164.2, 84.8)
- moved J801 3.00 mm to (146.5, 78.3)
- moved U901 3.00 mm to (149.3, 84.8)
- moved U902 3.00 mm to (145.2, 84.8)
- moved J601 2.00 mm to (127.5, 78.3)
- moved U701 2.00 mm to (130.3, 84.8)
- moved U702 2.00 mm to (126.2, 84.8)
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Routing:
- net GND: vias 93 -> 91
Other:
- board size 153.4 x 20.8 mm -> 147.5 x 20.8 mm
